File: DCDC33V.sch (KiCad schematic (older format))
At the start: 5 parts, among them U3 TL2575

Commit message: Layout 0.02
Connections:
- net 33Out: now reaches D2.2 (K), L2.1, U3.2 (OUTPUT)
Changed lines of the file:
@@
-EESchema Schematic File Version 2  date 26/04/2014 12:34:29
+EESchema Schematic File Version 2  date 26/04/2014 16:22:01
 LIBS:power
 LIBS:device
@@
 Gnd
 Connection ~ 4600 5000
+Text Label 5700 4300 0    60   ~ 0
+33Out
+Text Label 5700 4250 0    60   ~ 0
+Out33
+Text Label 5450 4300 0    60   ~ 0
+Out33
 $EndSCHEMATC
