File: blipr.kicad_pcb (KiCad board)
At the start: 2 copper layers, 13 parts, among them U1 AY-3-8910, U2 LM2575S, U3 TL2575, U4 RN42, U5 SN74LVC8T245DGVR

Commit message: Layout 0.02
Parts:
- added 21DC: VAL**, 21DC, B.Cu at (105.0, 126.0)
- added HD3x2SMD: VAL**, HD3x2SMD, F.Cu at (164.5, 161.0)
- added K1: CONN_3, 21DC, F.Cu at (96.0, 126.5)
- added P1: CONN_3X2, HD3x2SMD, F.Cu at (138.5, 185.5)
- added U6: FT231XS, SSOP20, F.Cu at (154.0, 161.5)
- added U7: ATXMEGA8E5, TQFP32, F.Cu at (184.5, 143.0)
- L1, L2: footprint SELF26 -> SMDSVP10
- U1: moved to B.Cu
- moved L2 64.2 mm to (124.0, 153.0)
- moved U1 62.3 mm to (170.0, 117.5), turned to 0 degrees
- moved C4 62.1 mm to (137.0, 149.0), turned to 90 degrees
- moved C2 61.3 mm to (137.0, 119.5)
- moved C3 61.2 mm to (105.5, 140.0)
- moved D1 59.9 mm to (113.5, 123.5), turned to 0 degrees
- moved C1 59.1 mm to (105.5, 111.0)
- moved U3 58.8 mm to (117.0, 143.5)
- moved D2 58.4 mm to (113.5, 153.0), turned to 0 degrees
- moved U2 57.2 mm to (117.0, 114.5)
- moved U5 48.2 mm to (162.0, 139.0), turned to 180 degrees
- moved U4 35.9 mm to (184.5, 166.0), turned to 180 degrees
- moved L1 24.9 mm to (124.0, 123.5)
Connections:
- U1 pad 30: N-0000016 -> N-0000050
- U1 pad 31: N-0000015 -> N-0000051
- U1 pad 32: N-0000014 -> N-0000052
- U1 pad 33: N-0000013 -> N-0000053
- U1 pad 34: N-0000012 -> (no net)
- U1 pad 35: N-0000040 -> (no net)
- U1 pad 36: N-0000043 -> (no net)
- U1 pad 37: N-0000046 -> (no net)
- U5 pad 10: N-0000016 -> (no net)
- U5 pad 3: N-0000046 -> N-0000050
- U5 pad 4: N-0000043 -> N-0000051
- U5 pad 5: N-0000040 -> N-0000052
- U5 pad 6: N-0000012 -> N-0000053
- U5 pad 7: N-0000013 -> (no net)
- U5 pad 8: N-0000014 -> (no net)
- U5 pad 9: N-0000015 -> (no net)
Routing:
- net DGND: track 0.00 -> 104.1 mm
- net +3.3V: track 0.00 -> 31.1 mm
- net +5V: track 0.00 -> 31.1 mm
- net +12V: track 0.00 -> 16.9 mm
- net N-0000050: track 0.00 -> 14.4 mm
- net N-00000137: track 0.00 -> 13.7 mm
- net N-0000051: track 0.00 -> 13.6 mm
- net N-00000136: track 0.00 -> 13.2 mm
- net N-0000052: track 0.00 -> 12.8 mm
- net N-0000053: track 0.00 -> 12.0 mm
- added copper zone on F.Cu, net DGND
Other:
- board outline added: 100 x 75 mm
- net class Power12 added: clearance 0.254, trace_width 1, via_dia 0.889, via_drill 0.635
- net class Power3 added: clearance 0.254, trace_width 1, via_dia 0.889, via_drill 0.635
- net class Power5 added: clearance 0.254, trace_width 1, via_dia 0.889, via_drill 0.635

Commit message: Layout 0.03
Parts:
- removed 21DC: VAL**, 21DC
- removed HD3x2SMD: VAL**, HD3x2SMD
- added C5: 47p, SM1206, F.Cu at (182.6, 163.2)
- added C6: 47p, SM1206, F.Cu at (187.3, 160.5)
- added C7: 100n, SM0603_Capa, F.Cu at (188.2, 157.2)
- added CON1: BARREL_JACK, BARREL_JACK, F.Cu at (194.6, 127.6)
- added D3: LED, LED-1206, F.Cu at (145.4, 162.7)
- added D4: LED, LED-1206, F.Cu at (145.4, 159.1)
- added P2: CONN_6, USB_MINI_B, F.Cu at (185.5, 170.6)
- added R1: 27, SM0603_Resistor, F.Cu at (185.0, 156.4)
- added R2: 27, SM0603_Resistor, F.Cu at (184.2, 158.2)
- added R3: 330, SM0603_Resistor, F.Cu at (149.6, 162.7)
- added R4: 330, SM0603_Resistor, F.Cu at (140.7, 159.1)
- added SM0603_resistor: Val**, SM0603_Resistor, F.Cu at (151.2, 137.0)
- added SM0603_resistor: Val**, SM0603_Resistor, F.Cu at (109.6, 132.2)
- C1, C2, C3, C4: footprint SMD403 -> CAP63
- K1: moved to B.Cu
- L1, L2: footprint SMDSVP10 -> MCB
- U5: footprint SSOP20 -> SSOP24
- moved P1 60.6 mm to (173.1, 135.8), turned to 90 degrees
- moved C1 40.0 mm to (105.4, 151.0), turned to 180 degrees
- moved U6 36.1 mm to (188.6, 151.3), turned to 180 degrees
- moved C3 29.0 mm to (105.4, 111.0), turned to 180 degrees
- moved U4 25.4 mm to (159.7, 160.5)
- moved U7 22.6 mm to (162.1, 139.8), turned to 180 degrees
- moved L2 12.8 mm to (121.6, 165.6)
- moved C4 11.2 mm to (126.8, 153.6), turned to 270 degrees
- moved U5 10.7 mm to (162.5, 128.3)
- moved C2 10.3 mm to (129.6, 112.4), turned to 270 degrees
- moved U3 10.0 mm to (117.0, 153.5)
- moved K1 9.30 mm to (104.4, 122.5)
- moved D2 7.59 mm to (111.8, 160.4)
- moved U1 7.01 mm to (170.4, 110.5)
- moved L1 2.60 mm to (126.6, 123.6)
Connections:
- net N-00000137 renamed /DCDC33V/33Out
- K1 pad 1: (no net) -> +12V
- K1 pad 2: (no net) -> DGND
- P1 pad 1: (no net) -> /PDI_DATA
- P1 pad 2: (no net) -> +3.3V
- P1 pad 5: (no net) -> /PDI_CLK
- P1 pad 6: (no net) -> DGND
- U1 pad 34: (no net) -> N-0000018
- U1 pad 35: (no net) -> N-0000017
- U1 pad 36: (no net) -> N-0000016
- U1 pad 37: (no net) -> N-0000015
- U1 pad 40: (no net) -> +5V
- U4 pad 1: (no net) -> DGND
- U4 pad 11: (no net) -> +3.3V
- U4 pad 12: (no net) -> DGND
- U4 pad 13: (no net) -> /RX
- U4 pad 14: (no net) -> /TX
- U4 pad 19: (no net) -> /PIO2
- U4 pad 22: (no net) -> /PIO5
- U4 pad 4: (no net) -> DGND
- U5 pad 10: (no net) -> N-0000015
- U5 pad 14: (no net) -> /BLIP0
- U5 pad 15: (no net) -> /BLIP1
- U5 pad 16: (no net) -> /BLIP2
- U5 pad 17: (no net) -> /BLIP3
- U5 pad 18: (no net) -> /BLIP4
- U5 pad 19: (no net) -> /BLIP5
- U5 pad 2: (no net) -> DGND
- U5 pad 20: (no net) -> /BLIP6
- U5 pad 7: (no net) -> N-0000018
- U5 pad 8: (no net) -> N-0000017
- U5 pad 9: (no net) -> N-0000016
- U6 pad 11: (no net) -> N-000005
- U6 pad 12: (no net) -> N-000006
- U6 pad 13: (no net) -> /FGND
- U6 pad 14: (no net) -> /FGND
- U6 pad 15: (no net) -> N-000003
- U6 pad 16: (no net) -> DGND
- U6 pad 3: (no net) -> +3.3V
- U6 pad 6: (no net) -> DGND
- U7 pad 1: (no net) -> DGND
- U7 pad 10: (no net) -> /BLIP6
- U7 pad 11: (no net) -> /BLIP5
- U7 pad 12: (no net) -> /BLIP4
- U7 pad 13: (no net) -> /BLIP3
- U7 pad 14: (no net) -> /BLIP2
- U7 pad 15: (no net) -> /BLIP1
- U7 pad 16: (no net) -> /BLIP0
- U7 pad 17: (no net) -> +3.3V
- U7 pad 18: (no net) -> DGND
- U7 pad 21: (no net) -> /TX
- U7 pad 22: (no net) -> /RX
- U7 pad 7: (no net) -> /PDI_DATA
- U7 pad 8: (no net) -> /PDI_CLK
- U7 pad 9: (no net) -> /BLIP7
Routing:
- net +3.3V: track 31.1 -> 178.9 mm
- net DGND: track 104.1 -> 215.4 mm
- net +12V: track 16.9 -> 57.7 mm
- net +5V: track 31.1 -> 71.6 mm
- net N-000003: track 0.00 -> 23.0 mm
- net /TX: track 0.00 -> 21.1 mm
- net /RX: track 0.00 -> 15.8 mm
- net /PDI_DATA: track 0.00 -> 11.8 mm
- net N-0000015: track 0.00 -> 11.4 mm
- net N-0000012: track 0.00 -> 10.9 mm
- net N-000001: track 0.00 -> 10.0 mm
- net N-0000016: track 0.00 -> 9.50 mm
- net N-0000017: track 0.00 -> 8.95 mm
- net N-0000018: track 0.00 -> 8.16 mm
- net N-000005: track 0.00 -> 7.65 mm
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Other:
- outline, holes or cut-outs redrawn
- net class Default: clearance 0.254 -> 0.1778
- net class Power12: clearance 0.254 -> 0.2032; trace_width 1 -> 0.3556
- net class Power3: clearance 0.254 -> 0.2032; trace_width 1 -> 0.3048
- net class Power5: clearance 0.254 -> 0.2032; trace_width 1 -> 0.3556
- rule trace_clearance: 0.254 -> 0.1778
